File: samples/placement-test.kicad_pcb (KiCad board)
At the start: 2 copper layers, 5 parts, among them T1 Through hole

Commit message: Release v0.1.1: MSI installer, BOM validation and description fixes
Other:
- board text added: "RevB"
Changed lines of the file:
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@@
   (general (thickness 1.6))
   (paper "A4")
-  (layers (0 "F.Cu" signal) (2 "B.Cu" signal))
+  (layers (0 "F.Cu" signal) (2 "B.Cu" signal) (5 "F.SilkS" user "F.Silkscreen"))
+  (gr_text "RevB" (at 15 20) (layer "F.SilkS") (effects (font (size 1 1) (thickness 0.15))))
   (setup (pad_to_mask_clearance 0) (aux_axis_origin 10 20)
     (pcbplotparams
